File: BClock.kicad_pcb (KiCad board)
At the start: 2 copper layers, 168.1 x 32 mm, 72 parts, among them J1 Conn_01x03_Pin, J2 Conn_01x03_Pin, U1 WS2811, U10 WS2811, U2 WS2811, U3 WS2811, U4 WS2811, U5 WS2811, U6 WS2811, U7 WS2811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

Commit message: NEW: Added ESP32C3 and level shifter
Parts:
- added J3: Conn_01x08_Socket, Connector_PinHeader_2.54mm:PinHeader_1x08_P2.54mm_Vertical, F.Cu at (170.2, 55.9)
- added J4: Conn_01x08_Socket, Connector_PinHeader_2.54mm:PinHeader_1x08_P2.54mm_Vertical, F.Cu at (170.7, 80.8)
- added J5: Conn_01x06_Socket, Connector_PinHeader_2.54mm:PinHeader_1x06_P2.54mm_Vertical, F.Cu at (202.7, 59.9)
- added U11: ESP32-C3_SUPERMINI, Mikes Library:MODULE_ESP32-C3_SUPERMINI, F.Cu at (160.5, 67.6)
- added U12: 74AHCT125, Package_DIP:DIP-14_W10.16mm, F.Cu at (120.4, 63.0)
- moved J1 8.80 mm to (76.7, 70.1)
- moved J2 8.26 mm to (229.6, 70.1)
Connections:
- net /ws2811/DIN renamed DATA_IN
- net VDD renamed 5V
Routing:
- net IN1: track 0.00 -> 62.3 mm
- net IN4: track 0.00 -> 61.8 mm
- net IN2: track 0.00 -> 58.4 mm
- net IN3: track 0.00 -> 54.8 mm
- net 5V: track 0.00 -> 45.6 mm, vias 0 -> 2
- net GND: track 154.1 -> 162.2 mm
- net Net-(J4-Pin_4): track 0.00 -> 5.70 mm
- net Net-(J4-Pin_8): track 0.00 -> 5.70 mm
- net Net-(J4-Pin_5): track 0.00 -> 5.70 mm
- net Net-(J4-Pin_3): track 0.00 -> 5.70 mm
- net /ws2820/DOUT: track 18.5 -> 24.0 mm
- net Net-(J3-Pin_6): track 0.00 -> 4.17 mm
- net Net-(J3-Pin_8): track 0.00 -> 4.17 mm
- net Net-(J3-Pin_7): track 0.00 -> 4.17 mm
- net Net-(J3-Pin_5): track 0.00 -> 4.17 mm
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Other:
- board size 168.1 x 32 mm -> 159.5 x 53.3 mm
