File: ws2811.kicad_sch (KiCad schematic)
At the start: 7 parts, among them U2 WS2811

Commit message: NEW: Added ESP32C3 and level shifter
Parts:
- renumbered C2 to C8, D4 to D22, D5 to D23, D6 to D24, R3 to R15, R4 to R16, U2 to U8
Changed lines of the file:
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@@
 		(dnp no)
 		(fields_autoplaced yes)
-		(property "Reference" "U2"
+		(property "Reference" "U8"
 			(at 105.0641 67.31 0)
 			(effects
@@
 		(dnp no)
 		(fields_autoplaced yes)
-		(property "Reference" "R4"
+		(property "Reference" "R16"
 			(at 105.41 58.4199 0)
 			(effects
@@
 		(dnp no)
 		(fields_autoplaced yes)
-		(property "Reference" "D5"
+		(property "Reference" "D23"
 			(at 115.2525 71.12 0)
 			(effects
@@
 		(dnp no)
 		(fields_autoplaced yes)
-		(property "Reference" "D6"
+		(property "Reference" "D24"
 			(at 115.2525 81.28 0)
 			(effects
@@
 		(dnp no)
 		(fields_autoplaced yes)
-		(property "Reference" "C2"
+		(property "Reference" "C8"
 			(at 92.71 58.42 90)
 			(effects
@@
 		(dnp no)
 		(fields_autoplaced yes)
-		(property "Reference" "D4"
+		(property "Reference" "D22"
 			(at 115.2525 59.69 0)
 			(effects
@@
 		(on_board yes)
 		(dnp no)
-		(property "Reference" "R3"
+		(property "Reference" "R15"
 			(at 88.9 68.58 90)
 			(effects
